Commit message: Linked laser & imu frame directly to base_link

File: buggy/urdf/buggy.urdf (robot description, URDF)
Before this commit: robot buggy_2d, 9 links, 8 joints
Links:
- removed link imu_link
- removed link laser_link
- added link imu; visual box size=0.057 0.042 0.023
- added link laser; visual cylinder length=0.09 radius=0.07
Joints:
- removed joint laser_link_joint
- added joint laser_joint: type fixed, parent base_link, child laser, origin xyz=-0.36 0 1.46
- joint imu_link_joint: child imu_link -> imu; origin xyz=0 0.036 -0.42 rpy=-1.57075 1.57075 0 -> xyz=-0.43 0.036 0.58 rpy=-1.57075 1.57075 0; parent beam -> base_link

Commit message: Re-positioned IMU

File: buggy/urdf/buggy.urdf (robot description, URDF)
Before this commit: robot buggy_2d, 9 links, 8 joints
Links:
- removed link imu
- added link front; visual box size=0.6 1.12 0.39
- added link imu_link; visual box size=0.057 0.042 0.023
- link base_link: geometry visual box size=2.43 1.12 0.09
- link beam: geometry visual box size=0.05 0.05 1.31
- link left_back_wheel: geometry visual cylinder length=0.22 radius=0.21
- link left_front_wheel: geometry visual cylinder length=0.22 radius=0.21
- link right_back_wheel: geometry visual cylinder length=0.22 radius=0.21
- link right_front_wheel: geometry visual cylinder length=0.22 radius=0.21
- link seat: geometry visual box size=1.1 1.12 0.39
Joints:
- added joint front_link_joint: type fixed, parent base_link, child front, origin xyz=0.93 0 0.24
- joint beam_link_joint: origin xyz=0 0 0.7 -> xyz=0 0 0.85435
- joint imu_link_joint: child imu -> imu_link; origin xyz=-0.43 0.036 0.58 rpy=-1.57075 1.57075 0 -> xyz=0.39 -0.47 0.05 rpy=0 0 0
- joint laser_joint: origin xyz=-0.36 0 1.46 -> xyz=-0.31 0 1.715
- joint left_back_wheel: origin xyz=-0.83 0.41 -0.15 rpy=0 0 0 -> xyz=-0.63 0.43 -0.05 rpy=0 0 0
- joint left_front_wheel: origin xyz=0.83 0.41 -0.15 rpy=0 0 0 -> xyz=1.02 0.43 -0.05 rpy=0 0 0
- joint right_back_wheel: origin xyz=-0.83 -0.41 -0.15 rpy=0 0 0 -> xyz=-0.63 -0.43 -0.05 rpy=0 0 0
- joint right_front_wheel: origin xyz=0.83 -0.41 -0.15 rpy=0 0 0 -> xyz=1.02 -0.43 -0.05 rpy=0 0 0
- joint seat_link_joint: origin xyz=-0.43 0 0.3 -> xyz=-0.35 0 0.24
